File: mini_chernobyl_dice_interface_pcb/mini_chernobyl_dice_interface_pcb.sch (KiCad schematic (older format))
At the start: 17 parts, among them SW1 SW_Push, SW2 ROTARY-ENCODER, U1 CC56-12EWA, U2 CC56-12EWA

Commit message: sync project; add firmware
Parts:
- added D5, D6, D7: LED_ALT, LED_THT:LED_D3.0mm_Horizontal_O1.27mm_Z2.0mm, symbol Device:LED_ALT
- added R6, R7, R8: R_Small, Resistor_THT:R_Axial_DIN0207_L6.3mm_D2.5mm_P10.16mm_Horizontal, symbol Device:R_Small
- D2, D3, D4: footprint LED_THT:LED_D3.0mm -> LED_THT:LED_D3.0mm_Horizontal_O1.27mm_Z2.0mm
Connections:
- net GND: now also D5.1 (K), D6.1 (K), D7.1 (K)
- net at H1.7 (UV), R3.2, R4.2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: now also R6.2, R7.2, R8.2
- new net: D5.2 (A), R6.1
- new net: D7.2 (A), R8.1
- new net: D6.2 (A), R7.1
Other:
- moved on the sheet: D2, D3, D4, R3, R4, R5
Changed lines of the file:
@@
 U 1 1 5E4FC5FD
 P 2750 5600
-F 0 "LS1" H 2950 5700 50  0000 L CNN
-F 1 "SPEAKER" H 2900 5800 50  0000 L CNN
+F 0 "LS1" H 2650 5400 50  0000 L CNN
+F 1 "SPEAKER" H 2350 5700 50  0000 L CNN
 F 2 "Buzzer_Beeper:Buzzer_TDK_PS1240P02BT_D12.2mm_H6.5mm" H 2750 5400 50  0001 C CNN
 F 3 "~" H 2740 5550 50  0001 C CNN
@@
 L Device:R_Small R3
 U 1 1 5E2E9382
-P 3350 5750
-F 0 "R3" V 3250 5700 50  0000 L CNN
-F 1 "R_Small" V 3250 5600 50  0001 L CNN
-F 2 "Resistor_THT:R_Axial_DIN0207_L6.3mm_D2.5mm_P10.16mm_Horizontal" H 3350 5750 50  0001 C CNN
-F 3 "~" H 3350 5750 50  0001 C CNN
-	1    3350 5750
+P 3350 5450
+F 0 "R3" V 3250 5400 50  0000 L CNN
+F 1 "R_Small" V 3250 5300 50  0001 L CNN
+F 2 "Resistor_THT:R_Axial_DIN0207_L6.3mm_D2.5mm_P10.16mm_Horizontal" H 3350 5450 50  0001 C CNN
+F 3 "~" H 3350 5450 50  0001 C CNN
+	1    3350 5450
 	0    1    1    0
 $EndComp
@@
 L Device:R_Small R5
 U 1 1 5E2E9A23
-P 3350 6150
-F 0 "R5" V 3250 6100 50  0000 L CNN
-F 1 "R_Small" V 3250 6000 50  0001 L CNN
-F 2 "Resistor_THT:R_Axial_DIN0207_L6.3mm_D2.5mm_P10.16mm_Horizontal" H 3350 6150 50  0001 C CNN
-F 3 "~" H 3350 6150 50  0001 C CNN
-	1    3350 6150
+P 3350 5850
+F 0 "R5" V 3250 5800 50  0000 L CNN
+F 1 "R_Small" V 3250 5700 50  0001 L CNN
+F 2 "Resistor_THT:R_Axial_DIN0207_L6.3mm_D2.5mm_P10.16mm_Horizontal" H 3350 5850 50  0001 C CNN
+F 3 "~" H 3350 5850 50  0001 C CNN
+	1    3350 5850
 	0    1    1    0
 $EndComp
@@
 L Device:R_Small R4
 U 1 1 5E2EA239
-P 3350 5950
-F 0 "R4" V 3250 5900 50  0000 L CNN
-F 1 "R_Small" V 3250 5800 50  0001 L CNN
-F 2 "Resistor_THT:R_Axial_DIN0207_L6.3mm_D2.5mm_P10.16mm_Horizontal" H 3350 5950 50  0001 C CNN
-F 3 "~" H 3350 5950 50  0001 C CNN
-	1    3350 5950
+P 3350 5650
+F 0 "R4" V 3250 5600 50  0000 L CNN
+F 1 "R_Small" V 3250 5500 50  0001 L CNN
+F 2 "Resistor_THT:R_Axial_DIN0207_L6.3mm_D2.5mm_P10.16mm_Horizontal" H 3350 5650 50  0001 C CNN
+F 3 "~" H 3350 5650 50  0001 C CNN
+	1    3350 5650
 	0    1    1    0
 $EndComp
@@
 L Device:LED_ALT D4
 U 1 1 5E2EBE25
-P 3600 6150
-F 0 "D4" H 3600 6250 50  0000 C CNN
-F 1 "LED_ALT" H 3593 6275 50  0001 C CNN
-F 2 "LED_THT:LED_D3.0mm" H 3600 6150 50  0001 C CNN
-F 3 "~" H 3600 6150 50  0001 C CNN
-	1    3600 6150
+P 3600 5850
+F 0 "D4" H 3600 5950 50  0000 C CNN
+F 1 "LED_ALT" H 3593 5975 50  0001 C CNN
+F 2 "LED_THT:LED_D3.0mm_Horizontal_O1.27mm_Z2.0mm" H 3600 5850 50  0001 C CNN
+F 3 "~" H 3600 5850 50  0001 C CNN
+	1    3600 5850
 	-1   0    0    -1
 $EndComp
@@
 L Device:LED_ALT D3
 U 1 1 5E2EB684
-P 3600 5950
-F 0 "D3" H 3600 6050 50  0000 C CNN
-F 1 "LED_ALT" H 3593 6075 50  0001 C CNN
-F 2 "LED_THT:LED_D3.0mm" H 3600 5950 50  0001 C CNN
-F 3 "~" H 3600 5950 50  0001 C CNN
-	1    3600 5950
+P 3600 5650
+F 0 "D3" H 3600 5750 50  0000 C CNN
+F 1 "LED_ALT" H 3593 5775 50  0001 C CNN
+F 2 "LED_THT:LED_D3.0mm_Horizontal_O1.27mm_Z2.0mm" H 3600 5650 50  0001 C CNN
+F 3 "~" H 3600 5650 50  0001 C CNN
+	1    3600 5650
 	-1   0    0    -1
 $EndComp
@@
 L Device:LED_ALT D2
 U 1 1 5E2EAB47
-P 3600 5750
-F 0 "D2" H 3600 5850 50  0000 C CNN
-F 1 "LED_ALT" H 3593 5875 50  0001 C CNN
-F 2 "LED_THT:LED_D3.0mm" H 3600 5750 50  0001 C CNN
-F 3 "~" H 3600 5750 50  0001 C CNN
-	1    3600 5750
+P 3600 5450
+F 0 "D2" H 3600 5550 50  0000 C CNN
+F 1 "LED_ALT" H 3593 5575 50  0001 C CNN
+F 2 "LED_THT:LED_D3.0mm_Horizontal_O1.27mm_Z2.0mm" H 3600 5450 50  0001 C CNN
+F 3 "~" H 3600 5450 50  0001 C CNN
+	1    3600 5450
 	-1   0    0    -1
 $EndComp
@@
 Wire Wire Line
 	2550 6000 2550 6100
-Wire Wire Line
-	3250 5750 3250 5950
-Connection ~ 3250 5950
-Wire Wire Line
-	3250 5950 3250 6150
-Wire Wire Line
-	3750 5750 3800 5750
-Wire Wire Line
-	3800 5750 3800 5950
-Wire Wire Line
-	3800 5950 3750 5950
-Wire Wire Line
-	3800 5950 3800 6150
-Wire Wire Line
-	3800 6150 3750 6150
-Connection ~ 3800 5950
 Wire Wire Line
 	3050 5050 2700 5050
@@
 Connection ~ 4050 5250
 Wire Wire Line
-	4050 5250 4050 5950
-Wire Wire Line
-	3800 5950 4050 5950
-Connection ~ 4050 5950
-Wire Wire Line
-	4050 5950 4050 6800
-Wire Wire Line
 	2450 6700 2450 6800
 Wire Wire Line
@@
 Wire Wire Line
 	4050 4450 4050 5250
-Text Notes 3650 5550 0    50   ~ 0
+Text Notes 4500 5500 0    50   ~ 0
 UV LEDS
 Text Notes 2350 6950 0    50   ~ 0
@@
 Text Notes 8600 2100 0    100  ~ 0
 7-SEGMENT DISPLAYS
+$Comp
+L Device:R_Small R6
+U 1 1 5EE08559
+P 3350 6050
+F 0 "R6" V 3250 6000 50  0000 L CNN
+F 1 "R_Small" V 3250 5900 50  0001 L CNN
+F 2 "Resistor_THT:R_Axial_DIN0207_L6.3mm_D2.5mm_P10.16mm_Horizontal" H 3350 6050 50  0001 C CNN
+F 3 "~" H 3350 6050 50  0001 C CNN
+	1    3350 6050
+	0    1    1    0
+$EndComp
+$Comp
+L Device:R_Small R8
+U 1 1 5EE0855F
+P 3350 6450
+F 0 "R8" V 3250 6400 50  0000 L CNN
+F 1 "R_Small" V 3250 6300 50  0001 L CNN
+F 2 "Resistor_THT:R_Axial_DIN0207_L6.3mm_D2.5mm_P10.16mm_Horizontal" H 3350 6450 50  0001 C CNN
+F 3 "~" H 3350 6450 50  0001 C CNN
+	1    3350 6450
+	0    1    1    0
+$EndComp
+$Comp
+L Device:R_Small R7
+U 1 1 5EE08565
+P 3350 6250
+F 0 "R7" V 3250 6200 50  0000 L CNN
+F 1 "R_Small" V 3250 6100 50  0001 L CNN
+F 2 "Resistor_THT:R_Axial_DIN0207_L6.3mm_D2.5mm_P10.16mm_Horizontal" H 3350 6250 50  0001 C CNN
+F 3 "~" H 3350 6250 50  0001 C CNN
+	1    3350 6250
+	0    1    1    0
+$EndComp
+$Comp
+L Device:LED_ALT D7
+U 1 1 5EE0856B
+P 3600 6450
+F 0 "D7" H 3600 6550 50  0000 C CNN
+F 1 "LED_ALT" H 3593 6575 50  0001 C CNN
+F 2 "LED_THT:LED_D3.0mm_Horizontal_O1.27mm_Z2.0mm" H 3600 6450 50  0001 C CNN
+F 3 "~" H 3600 6450 50  0001 C CNN
+	1    3600 6450
+	-1   0    0    -1
+$EndComp
+$Comp
+L Device:LED_ALT D6
+U 1 1 5EE08571
+P 3600 6250
+F 0 "D6" H 3600 6350 50  0000 C CNN
+F 1 "LED_ALT" H 3593 6375 50  0001 C CNN
+F 2 "LED_THT:LED_D3.0mm_Horizontal_O1.27mm_Z2.0mm" H 3600 6250 50  0001 C CNN
+F 3 "~" H 3600 6250 50  0001 C CNN
+	1    3600 6250
+	-1   0    0    -1
+$EndComp
+$Comp
+L Device:LED_ALT D5
+U 1 1 5EE08577
+P 3600 6050
+F 0 "D5" H 3600 6150 50  0000 C CNN
+F 1 "LED_ALT" H 3593 6175 50  0001 C CNN
+F 2 "LED_THT:LED_D3.0mm_Horizontal_O1.27mm_Z2.0mm" H 3600 6050 50  0001 C CNN
+F 3 "~" H 3600 6050 50  0001 C CNN
+	1    3600 6050
+	-1   0    0    -1
+$EndComp
+Wire Wire Line
+	3250 5450 3250 5650
+Connection ~ 3250 5650
+Wire Wire Line
+	3250 5650 3250 5850
+Connection ~ 3250 5850
+Wire Wire Line
+	3250 5850 3250 5950
+Connection ~ 3250 5950
+Wire Wire Line
+	3250 5950 3250 6050
+Connection ~ 3250 6050
+Wire Wire Line
+	3250 6050 3250 6250
+Connection ~ 3250 6250
+Wire Wire Line
+	3250 6250 3250 6450
+Wire Wire Line
+	4050 5250 4050 5950
+Wire Wire Line
+	3750 5450 3800 5450
+Wire Wire Line
+	3800 5450 3800 5650
+Wire Wire Line
+	3800 6450 3750 6450
+Wire Wire Line
+	3750 5650 3800 5650
+Connection ~ 3800 5650
+Wire Wire Line
+	3800 5650 3800 5850
+Wire Wire Line
+	3750 5850 3800 5850
+Connection ~ 3800 5850
+Wire Wire Line
+	3800 5850 3800 5950
+Wire Wire Line
+	3750 6050 3800 6050
+Connection ~ 3800 6050
+Wire Wire Line
+	3800 6050 3800 6250
+Wire Wire Line
+	3750 6250 3800 6250
+Connection ~ 3800 6250
+Wire Wire Line
+	3800 6250 3800 6450
+Wire Wire Line
+	3800 5950 4050 5950
+Connection ~ 3800 5950
+Wire Wire Line
+	3800 5950 3800 6050
+Connection ~ 4050 5950
+Wire Wire Line
+	4050 5950 4050 6800
 $EndSCHEMATC
